File: LED/LED.kicad_pcb (KiCad board)
At the start: 2 copper layers, 72.4 x 72.4 mm, 17 parts, among them J1 JST_header

Commit message: Update after DRC checks, add extra switches for mini hakkero
Routing:
- net /SW_+: track 311.5 -> 308.0 mm
Other:
- board text added: "The present is me, da ze~"
