File: Unified/Unified.kicad_sch (KiCad schematic)
At the start: 57 parts, among them J1 USB_C_Receptacle_USB2.0_16P, J10 JST_switch_1, J11 JST_switch_2, J12 Conn_touch_1, J13 Conn_touch_2, J14 Bat_pos_sel, J15 Bat_neg_sel, J16 Conn_01x02, J17 Conn_01x07, J2 JST_battery, J3 JST_header, J4 JST_speaker, J5 JST_debug_swd, J6 JST_debug_serial, Q1 AO3401A, Q2 AO3400A, SW1 SW_power, U1 MCP73831-2-OT, U2 MAX98357A

Commit message: Add ground connection for MAX98357 pad, rewire GAIN and SD pins for header breakout, curse all actual EE nerds
Connections:
- net GND: now also U2.17 (PAD)
- net SPEAKER_GAIN: now also J17.4 (Pin_4)
- net SPEAKER_SD: now reaches A1.9 (GPIO6)
- net SPEAKER_SD: now also J17.5 (Pin_5), U2.4 (~{SD_MODE})
- no-connect marks 27 -> 22
Changed lines of the file:
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@@
 	)
 	(no_connect
-		(at 265.43 114.3)
-	)
-	(no_connect
 		(at 52.07 59.69)
 	)
@@
 	)
 	(no_connect
-		(at 146.05 162.56)
-	)
-	(no_connect
 		(at 29.21 67.31)
 	)
@@
 	)
 	(no_connect
-		(at 265.43 116.84)
-	)
-	(no_connect
 		(at 259.08 229.87)
 	)
@@
 	)
 	(no_connect
-		(at 100.33 167.64)
+		(at 265.43 124.46)
 	)
 	(no_connect
@@
 	)
 	(no_connect
-		(at 265.43 124.46)
-	)
-	(no_connect
-		(at 146.05 165.1)
-	)
-	(no_connect
 		(at 265.43 96.52)
 	)
 	(no_connect
-		(at 85.09 157.48)
+		(at 265.43 114.3)
 	)
 	(no_connect
@@
 	(wire
 		(pts
+			(xy 142.24 162.56) (xy 146.05 162.56)
+		)
+		(stroke
+			(width 0)
+			(type default)
+		)
+	)
+	(wire
+		(pts
 			(xy 226.06 222.25) (xy 226.06 219.71)
 		)
@@
 	(wire
 		(pts
+			(xy 82.55 157.48) (xy 85.09 157.48)
+		)
+		(stroke
+			(width 0)
+			(type default)
+		)
+	)
+	(wire
+		(pts
 			(xy 129.54 35.56) (xy 142.24 35.56)
 		)
@@
 	(wire
 		(pts
+			(xy 100.33 167.64) (xy 100.33 171.45)
+		)
+		(stroke
+			(width 0)
+			(type default)
+		)
+	)
+	(wire
+		(pts
 			(xy 171.45 109.22) (xy 167.64 109.22)
 		)
@@
 	(wire
 		(pts
+			(xy 261.62 116.84) (xy 265.43 116.84)
+		)
+		(stroke
+			(width 0)
+			(type default)
+		)
+	)
+	(wire
+		(pts
 			(xy 142.24 138.43) (xy 146.05 138.43)
 		)
@@
 	(wire
 		(pts
+			(xy 142.24 165.1) (xy 146.05 165.1)
+		)
+		(stroke
+			(width 0)
+			(type default)
+		)
+	)
+	(wire
+		(pts
 			(xy 99.06 237.49) (xy 99.06 240.03)
 		)
@@
 		)
 	)
+	(label "SPEAKER_SD"
+		(at 142.24 165.1 180)
+		(effects
+			(font
+				(size 1.27 1.27)
+			)
+			(justify right bottom)
+		)
+	)
 	(label "USB_VBUS"
 		(at 78.74 93.98 180)
@@
 		)
 	)
+	(label "SPEAKER_SD"
+		(at 261.62 116.84 180)
+		(effects
+			(font
+				(size 1.27 1.27)
+			)
+			(justify right bottom)
+		)
+	)
 	(label "SW_+"
 		(at 97.79 137.16 90)
@@
 		)
 	)
+	(label "SPEAKER_GAIN"
+		(at 142.24 162.56 180)
+		(effects
+			(font
+				(size 1.27 1.27)
+			)
+			(justify right bottom)
+		)
+	)
 	(label "BUTTON_4"
 		(at 261.62 134.62 180)
@@
 		)
 	)
+	(label "BAT_-"
+		(at 100.33 171.45 270)
+		(effects
+			(font
+				(size 1.27 1.27)
+			)
+			(justify right bottom)
+		)
+	)
 	(label "BUTTON_4"
 		(at 115.57 110.49 180)
@@
 		(effects
 			(font
+				(size 1.27 1.27)
+			)
+			(justify right bottom)
+		)
+	)
+	(label "SPEAKER_SD"
+		(at 82.55 157.48 180)
+		(effects
+			(font
